Commit message: Naming Convention
Fix variables names and convert taps to spaces.

File: urdf/box.urdf.xacro (robot description, xacro)
@@ -1,172 +1,172 @@
 <robot name="plane" xmlns:xacro="http://www.ros.org/wiki/xacro">
-	<link name="body">
-		<visual>
-			<geometry>
-				<box size="2 1 0.5" />
-			</geometry>
-		</visual>
-		<collision>
-			<geometry>
-				<box size="2 1 0.5" />
-			</geometry>
-		</collision>
-		<inertial>
-			<mass value="2" />
-			<inertia ixx="1.04166666666666" ixy="0" ixz="0" iyz="0"
-				iyy="3.5416666666666" izz="4.166666666666666" />
-		</inertial>
-	</link>
+    <link name="body">
+        <visual>
+            <geometry>
+                <box size="2 1 0.5" />
+            </geometry>
+        </visual>
+        <collision>
+            <geometry>
+                <box size="2 1 0.5" />
+            </geometry>
+        </collision>
+        <inertial>
+            <mass value="2" />
+            <inertia ixx="1.04166666666666" ixy="0" ixz="0" iyz="0"
+                iyy="3.5416666666666" izz="4.166666666666666" />
+        </inertial>
+    </link>
     ----------------------------------------------------------------------------  wheels
-	---------------------------------------------------------------------------front wheels
-	<link name="wheel_base_front">
-		<visual>
-			<geometry>
-				<box size="0.05 2 0.05" />
-			</geometry>
-		</visual>
-		<collision>
-			<geometry>
-				<box size="0.05 2 0.05" />
-			</geometry>
-		</collision>
-		<inertial>
-			<mass value="0.1" />
-			<inertia ixx="0.033354166666" ixy="0" ixz="0" iyz="0"
-				iyy=" 0.00004166666" izz="0.033354166666" />
-		</inertial>
-	</link>
-	<joint name=" body_to_wheel_base_front" type="fixed">
-		<origin xyz="1 0 -0.25" rpy="0 0 0" />
-		<parent link="body" />
-		<child link="wheel_base_front" />
-	</joint>
-	<link name="wheel_base_rear">
-		<visual>
-			<geometry>
-				<box size="0.05 2 0.05" />
-			</geometry>
-		</visual>
-		<collision>
-			<geometry>
-				<box size="0.05 2 0.05" />
-			</geometry>
-		</collision>
-		<inertial>
-			<mass value="0.1" />
-			<inertia ixx="0.033354166666" ixy="0" ixz="0" iyz="0"
-				iyy=" 0.00004166666" izz="0.033354166666" />
-		</inertial>
-	</link>
-	<joint name=" body_to_wheel_rear" type="fixed">
-		<origin xyz="-1 0 -0.25" rpy="0 0 0" />
-		<parent link="body" />
-		<child link="wheel_base_rear" />
-	</joint>
-	<link name="left_wheel_front">
-		<visual>
-			<origin xyz="0 0 0.05" />
-			<geometry>
-				<cylinder radius="0.3" length="0.1" />
-			</geometry>
-		</visual>
-		<collision>
-			<origin xyz="0 0 0.05" />
-			<geometry>
-				<cylinder radius="0.3" length="0.1" />
-			</geometry>
-		</collision>
-		<inertial>
-			<origin xyz="0 0 0.05" />
-			<mass value="0.1" />
-			<inertia ixx="0.0023333333333333" ixy="0" ixz="0" iyz="0"
-				iyy=" 0.0023333333333333" izz="0.00075" />
-		</inertial>
-	</link>
-	<joint name=" wheel_base_to_left_wheel_front" type="continuous">
-		<origin xyz="0 -1 0" rpy="1.57 0 0" />
-		<parent link="wheel_base_front" />
-		<child link="left_wheel_front" />
-		<axis xyz=" 0 0 1" />
-	</joint>
-	<link name="right_wheel_front">
-		<visual>
-			<origin xyz="0 0 -0.05" />
-			<geometry>
-				<cylinder radius="0.3" length="0.1" />
-			</geometry>
-		</visual>
-		<collision>
-			<origin xyz="0 0 -0.05" />
-			<geometry>
-				<cylinder radius="0.3" length="0.1" />
-			</geometry>
-		</collision>
-		<inertial>
-			<origin xyz="0 0 -0.05" />
-			<mass value="0.1" />
-			<inertia ixx="0.0023333333333333" ixy="0" ixz="0" iyz="0"
-				iyy=" 0.0023333333333333" izz="0.00075" />
-		</inertial>
-	</link>
-	<joint name=" wheel_base_to_right_wheel_front" type="continuous">
-		<origin xyz="0 1 0" rpy="1.57 0 0" />
-		<parent link="wheel_base_front" />
-		<child link="right_wheel_front" />
-		<axis xyz=" 0 0 1" />
-	</joint>
-	--
-	<link name="left_wheel_rear">
-		<visual>
-			<origin xyz="0 0 0.05" />
-			<geometry>
-				<cylinder radius="0.3" length="0.1" />
-			</geometry>
-		</visual>
-		<collision>
-			<origin xyz="0 0 0.05" />
-			<geometry>
-				<cylinder radius="0.3" length="0.1" />
-			</geometry>
-		</collision>
-		<inertial>
-			<origin xyz="0 0 0.05" />
-			<mass value="0.1" />
-			<inertia ixx="0.0023333333333333" ixy="0" ixz="0" iyz="0"
-				iyy=" 0.0023333333333333" izz="0.00075" />
-		</inertial>
-	</link>
-	<joint name=" wheel_base_to_left_wheel_rear" type="continuous">
-		<origin xyz="0 -1 0" rpy="1.57 0 0" />
-		<parent link="wheel_base_rear" />
-		<child link="left_wheel_rear" />
-		<axis xyz=" 0 0 1" />
-	</joint>
-	<link name="right_wheel_rear">
-		<visual>
-			<origin xyz="0 0 -0.05" />
-			<geometry>
-				<cylinder radius="0.3" length="0.1" />
-			</geometry>
-		</visual>
-		<collision>
-			<origin xyz="0 0 -0.05" />
-			<geometry>
-				<cylinder radius="0.3" length="0.1" />
-			</geometry>
-		</collision>
-		<inertial>
-			<origin xyz="0 0 -0.05" />
-			<mass value="0.1" />
-			<inertia ixx="0.0023333333333333" ixy="0" ixz="0" iyz="0"
-				iyy=" 0.0023333333333333" izz="0.00075" />
-		</inertial>
-	</link>
-	<joint name=" wheel_base_to_right_wheel_rear" type="continuous">
-		<origin xyz="0 1 0" rpy="1.57 0 0" />
-		<parent link="wheel_base_rear" />
-		<child link="right_wheel_rear" />
-		<axis xyz=" 0 0 1" />
-	</joint>
-	<gazebo>
+    ---------------------------------------------------------------------------front wheels
+    <link name="wheel_base_front">
+        <visual>
+            <geometry>
+                <box size="0.05 2 0.05" />
+            </geometry>
+        </visual>
+        <collision>
+            <geometry>
+                <box size="0.05 2 0.05" />
+            </geometry>
+        </collision>
+        <inertial>
+            <mass value="0.1" />
+            <inertia ixx="0.033354166666" ixy="0" ixz="0" iyz="0"
+                iyy=" 0.00004166666" izz="0.033354166666" />
+        </inertial>
+    </link>
+    <joint name=" body_to_wheel_base_front" type="fixed">
+        <origin xyz="1 0 -0.25" rpy="0 0 0" />
+        <parent link="body" />
+        <child link="wheel_base_front" />
+    </joint>
+    <link name="wheel_base_rear">
+        <visual>
+            <geometry>
+                <box size="0.05 2 0.05" />
+            </geometry>
+        </visual>
+        <collision>
+            <geometry>
+                <box size="0.05 2 0.05" />
+            </geometry>
+        </collision>
+        <inertial>
+            <mass value="0.1" />
+            <inertia ixx="0.033354166666" ixy="0" ixz="0" iyz="0"
+                iyy=" 0.00004166666" izz="0.033354166666" />
+        </inertial>
+    </link>
+    <joint name=" body_to_wheel_rear" type="fixed">
+        <origin xyz="-1 0 -0.25" rpy="0 0 0" />
+        <parent link="body" />
+        <child link="wheel_base_rear" />
+    </joint>
+    <link name="left_wheel_front">
+        <visual>
+            <origin xyz="0 0 0.05" />
+            <geometry>
+                <cylinder radius="0.3" length="0.1" />
+            </geometry>
+        </visual>
+        <collision>
+            <origin xyz="0 0 0.05" />
+            <geometry>
+                <cylinder radius="0.3" length="0.1" />
+            </geometry>
+        </collision>
+        <inertial>
+            <origin xyz="0 0 0.05" />
+            <mass value="0.1" />
+            <inertia ixx="0.0023333333333333" ixy="0" ixz="0" iyz="0"
+                iyy=" 0.0023333333333333" izz="0.00075" />
+        </inertial>
+    </link>
+    <joint name=" wheel_base_to_left_wheel_front" type="continuous">
+        <origin xyz="0 -1 0" rpy="1.57 0 0" />
+        <parent link="wheel_base_front" />
+        <child link="left_wheel_front" />
+        <axis xyz=" 0 0 1" />
+    </joint>
+    <link name="right_wheel_front">
+        <visual>
+            <origin xyz="0 0 -0.05" />
+            <geometry>
+                <cylinder radius="0.3" length="0.1" />
+            </geometry>
+        </visual>
+        <collision>
+            <origin xyz="0 0 -0.05" />
+            <geometry>
+                <cylinder radius="0.3" length="0.1" />
+            </geometry>
+        </collision>
+        <inertial>
+            <origin xyz="0 0 -0.05" />
+            <mass value="0.1" />
+            <inertia ixx="0.0023333333333333" ixy="0" ixz="0" iyz="0"
+                iyy=" 0.0023333333333333" izz="0.00075" />
+        </inertial>
+    </link>
+    <joint name=" wheel_base_to_right_wheel_front" type="continuous">
+        <origin xyz="0 1 0" rpy="1.57 0 0" />
+        <parent link="wheel_base_front" />
+        <child link="right_wheel_front" />
+        <axis xyz=" 0 0 1" />
+    </joint>
+    --
+    <link name="left_wheel_rear">
+        <visual>
+            <origin xyz="0 0 0.05" />
+            <geometry>
+                <cylinder radius="0.3" length="0.1" />
+            </geometry>
+        </visual>
+        <collision>
+            <origin xyz="0 0 0.05" />
+            <geometry>
+                <cylinder radius="0.3" length="0.1" />
+            </geometry>
+        </collision>
+        <inertial>
+            <origin xyz="0 0 0.05" />
+            <mass value="0.1" />
+            <inertia ixx="0.0023333333333333" ixy="0" ixz="0" iyz="0"
+                iyy=" 0.0023333333333333" izz="0.00075" />
+        </inertial>
+    </link>
+    <joint name=" wheel_base_to_left_wheel_rear" type="continuous">
+        <origin xyz="0 -1 0" rpy="1.57 0 0" />
+        <parent link="wheel_base_rear" />
+        <child link="left_wheel_rear" />
+        <axis xyz=" 0 0 1" />
+    </joint>
+    <link name="right_wheel_rear">
+        <visual>
+            <origin xyz="0 0 -0.05" />
+            <geometry>
+                <cylinder radius="0.3" length="0.1" />
+            </geometry>
+        </visual>
+        <collision>
+            <origin xyz="0 0 -0.05" />
+            <geometry>
+                <cylinder radius="0.3" length="0.1" />
+            </geometry>
+        </collision>
+        <inertial>
+            <origin xyz="0 0 -0.05" />
+            <mass value="0.1" />
+            <inertia ixx="0.0023333333333333" ixy="0" ixz="0" iyz="0"
+                iyy=" 0.0023333333333333" izz="0.00075" />
+        </inertial>
+    </link>
+    <joint name=" wheel_base_to_right_wheel_rear" type="continuous">
+        <origin xyz="0 1 0" rpy="1.57 0 0" />
+        <parent link="wheel_base_rear" />
+        <child link="right_wheel_rear" />
+        <axis xyz=" 0 0 1" />
+    </joint>
+    <gazebo>
     <plugin name="model_plugin" filename="libmodel_plugin.so"/>
   </gazebo>

File: urdf/plane.urdf.xacro (robot description, xacro)
@@ -1,196 +1,196 @@
 <robot name="plane" xmlns:xacro="http://www.ros.org/wiki/xacro">
-	<link name="body">
-		<visual>
-			<origin rpy="0 -1.57 0 " />
-			<geometry>
-				<cylinder radius="0.5" length="2.5" />
-			</geometry>
-		</visual>
-		<collision>
-			<origin rpy="0 -1.57 0 " />
-			<geometry>
-				<cylinder radius="0.5" length="2.5" />
-			</geometry>
-		</collision>
-		<inertial>
-			<origin rpy="0 -1.57 0 " />
-			<mass value="0.2" />
-			<inertia ixx="0.116666666666" ixy="0" ixz="0" iyz="0"
-				iyy="0.116666666666" izz="0.00416666666666" />
-		</inertial>
-	</link>
+    <link name="body">
+        <visual>
+            <origin rpy="0 -1.57 0 " />
+            <geometry>
+                <cylinder radius="0.5" length="2.5" />
+            </geometry>
+        </visual>
+        <collision>
+            <origin rpy="0 -1.57 0 " />
+            <geometry>
+                <cylinder radius="0.5" length="2.5" />
+            </geometry>
+        </collision>
+        <inertial>
+            <origin rpy="0 -1.57 0 " />
+            <mass value="0.2" />
+            <inertia ixx="0.116666666666" ixy="0" ixz="0" iyz="0"
+                iyy="0.116666666666" izz="0.00416666666666" />
+        </inertial>
+    </link>
     ----------------------------------------------------------------------------  wings
-	<link name="airfoil">
-		<visual>
-			<geometry>
-				<box size="0.5 6 0.1" />
-			</geometry>
-		</visual>
-		<collision>
-			<geometry>
-				<box size="0.5 6 0.1" />
-			</geometry>
-		</collision>
-		<inertial>
-			<mass value="2" />
-			<inertia ixx="6.0016666666666" ixy="0" ixz="0" iyz="0"
-				iyy="0.04333333333333" izz="6.0416666666666" />
-		</inertial>
-	</link>
-	<joint name="bodyToWing" type="revolute">
-		<origin xyz="0 0 0.4" rpy ="0 0 0"/>
-		<parent link="body" />
-		<child link="airfoil" />
-		<limit effort="1000.0" lower="-0.000872665" upper="0.000872665" velocity="0.5"/>
-	</joint>
+    <link name="airfoil">
+        <visual>
+            <geometry>
+                <box size="0.5 6 0.1" />
+            </geometry>
+        </visual>
+        <collision>
+            <geometry>
+                <box size="0.5 6 0.1" />
+            </geometry>
+        </collision>
+        <inertial>
+            <mass value="2" />
+            <inertia ixx="6.0016666666666" ixy="0" ixz="0" iyz="0"
+                iyy="0.04333333333333" izz="6.0416666666666" />
+        </inertial>
+    </link>
+    <joint name="bodyToWing" type="revolute">
+        <origin xyz="0 0 0.4" rpy ="0 0 0"/>
+        <parent link="body" />
+        <child link="airfoil" />
+        <limit effort="1000.0" lower="-0.000872665" upper="0.000872665" velocity="0.5"/>
+    </joint>
  -----------------------------------------------------------------------------------propeller
-	<link name="arm">
-		<visual>
-			<origin xyz="0 0 0.1" />
-			<geometry>
-				<cylinder radius="0.1" length="0.2" />
-			</geometry>
-		</visual>
-		<collision>
-			<origin xyz="0 0 0.1" />
-			<geometry>
-				<cylinder radius="0.1" length="0.2" />
-			</geometry>
-		</collision>
-		<inertial>
-			<origin xyz="0 0 0.1" />
-			<mass value="0.1" />
-			<inertia ixx="0.000583333" ixy="0" ixz="0" iyz="0"
-				iyy="0.000583333" izz="0.00008333333" />
-		</inertial>
-	</link>
-	<joint name="body_to_arm" type="continuous">
-		<origin xyz="1.25 0 0" rpy="0 1.57  0" />
-		<axis xyz="0 0 1" />
-		<parent link="body" />
-		<child link="arm" />
-	</joint>
-	<link name="propeller">
-		<visual>
-			<geometry>
-				<box size="0.8 0.2 0.05" />
-			</geometry>
-		</visual>
-		<collision>
-			<geometry>
-				<box size="0.8 0.2 0.05" />
-			</geometry>
-		</collision>
-		<inertial>
-			<mass value="0.1" />
-			<inertia ixx="0.00035416666666" ixy="0" ixz="0" iyz="0"
-				iyy=" 0.005354166666666" izz="0.005666666666" />
-		</inertial>
-	</link>
-	<joint name="arm_to_propeller" type="fixed">
-		<origin xyz="0 0 0.2" rpy="0 0 0" />
-		<parent link="arm" />
-		<child link="propeller" />
-	</joint>
+    <link name="arm">
+        <visual>
+            <origin xyz="0 0 0.1" />
+            <geometry>
+                <cylinder radius="0.1" length="0.2" />
+            </geometry>
+        </visual>
+        <collision>
+            <origin xyz="0 0 0.1" />
+            <geometry>
+                <cylinder radius="0.1" length="0.2" />
+            </geometry>
+        </collision>
+        <inertial>
+            <origin xyz="0 0 0.1" />
+            <mass value="0.1" />
+            <inertia ixx="0.000583333" ixy="0" ixz="0" iyz="0"
+                iyy="0.000583333" izz="0.00008333333" />
+        </inertial>
+    </link>
+    <joint name="body_to_arm" type="continuous">
+        <origin xyz="1.25 0 0" rpy="0 1.57  0" />
+        <axis xyz="0 0 1" />
+        <parent link="body" />
+        <child link="arm" />
+    </joint>
+    <link name="propeller">
+        <visual>
+            <geometry>
+                <box size="0.8 0.2 0.05" />
+            </geometry>
+        </visual>
+        <collision>
+            <geometry>
+                <box size="0.8 0.2 0.05" />
+            </geometry>
+        </collision>
+        <inertial>
+            <mass value="0.1" />
+            <inertia ixx="0.00035416666666" ixy="0" ixz="0" iyz="0"
+                iyy=" 0.005354166666666" izz="0.005666666666" />
+        </inertial>
+    </link>
+    <joint name="arm_to_propeller" type="fixed">
+        <origin xyz="0 0 0.2" rpy="0 0 0" />
+        <parent link="arm" />
+        <child link="propeller" />
+    </joint>
      ---------------------------------------------------------------------------front wheels
-	<link name="wheel_base">
-		<visual>
-			<geometry>
-				<box size="0.05 2 0.05" />
-			</geometry>
-		</visual>
-		<collision>
-			<geometry>
-				<box size="0.05 2 0.05" />
-			</geometry>
-		</collision>
-		<inertial>
-			<mass value="0.1" />
-			<inertia ixx="0.033354166666" ixy="0" ixz="0" iyz="0"
-				iyy=" 0.00004166666" izz="0.033354166666" />
-		</inertial>
-	</link>
-	<joint name=" body_to_wheel_base" type="fixed">
-		<origin xyz="1 0 -0.5" rpy="0 0 0" />
-		<parent link="body" />
-		<child link="wheel_base" />
-	</joint>
-	<link name="left_wheel">
-		<visual>
-			<origin xyz="0 0 0.05" />
-			<geometry>
-				<cylinder radius="0.3" length="0.1" />
-			</geometry>
-		</visual>
-		<collision>
-			<origin xyz="0 0 0.05" />
-			<geometry>
-				<cylinder radius="0.3" length="0.1" />
-			</geometry>
-		</collision>
-		<inertial>
-			<origin xyz="0 0 0.05" />
-			<mass value="0.1" />
-			<inertia ixx="0.0023333333333333" ixy="0" ixz="0" iyz="0"
-				iyy=" 0.0023333333333333" izz="0.00075" />
-		</inertial>
-	</link>
-	<joint name=" wheel_base_to_left_wheel" type="continuous">
-		<origin xyz="0 -1 0" rpy="1.57 0 0" />
-		<parent link="wheel_base" />
-		<child link="left_wheel" />
-		<axis xyz=" 0 0 1" />
-	</joint>
-	<link name="right_wheel">
-		<visual>
-			<origin xyz="0 0 -0.05" />
-			<geometry>
-				<cylinder radius="0.3" length="0.1" />
-			</geometry>
-		</visual>
-		<collision>
-			<origin xyz="0 0 -0.05" />
-			<geometry>
-				<cylinder radius="0.3" length="0.1" />
-			</geometry>
-		</collision>
-		<inertial>
-			<origin xyz="0 0 -0.05" />
-			<mass value="0.1" />
-			<inertia ixx="0.0023333333333333" ixy="0" ixz="0" iyz="0"
-				iyy=" 0.0023333333333333" izz="0.00075" />
-		</inertial>
-	</link>
-	<joint name=" wheel_base_to_right_wheel" type="continuous">
-		<origin xyz="0 1 0" rpy="1.57 0 0" />
-		<parent link="wheel_base" />
-		<child link="right_wheel" />
-		<axis xyz=" 0 0 1" />
-	</joint>
-	------------------------------------------------------------------------------------ rear sphere wheel
-	<link name="rear_wheel">
-		<visual>
-			<geometry>
-				<sphere radius="0.1" />
-			</geometry>
-		</visual>
-		<collision>
-			<geometry>
-				<sphere radius="0.1" />
-			</geometry>
-		</collision>
-		<inertial>
-			<mass value="0.1" />
-			<inertia ixx="0.0004" ixy="0" ixz="0" iyz="0"
-				iyy=" 0.0004" izz="0.0004" />
-		</inertial>
-	</link>
-	<joint name="body_to_rear_wheel" type="continuous">
-		<origin xyz="-1 0 -0.5" />
-		<axis xyz="0 1 0"/>
-		<parent link="body" />
-		<child link="rear_wheel" />
-	</joint>
-	<gazebo>
+    <link name="wheel_base">
+        <visual>
+            <geometry>
+                <box size="0.05 2 0.05" />
+            </geometry>
+        </visual>
+        <collision>
+            <geometry>
+                <box size="0.05 2 0.05" />
+            </geometry>
+        </collision>
+        <inertial>
+            <mass value="0.1" />
+            <inertia ixx="0.033354166666" ixy="0" ixz="0" iyz="0"
+                iyy=" 0.00004166666" izz="0.033354166666" />
+        </inertial>
+    </link>
+    <joint name=" body_to_wheel_base" type="fixed">
+        <origin xyz="1 0 -0.5" rpy="0 0 0" />
+        <parent link="body" />
+        <child link="wheel_base" />
+    </joint>
+    <link name="left_wheel">
+        <visual>
+            <origin xyz="0 0 0.05" />
+            <geometry>
+                <cylinder radius="0.3" length="0.1" />
+            </geometry>
+        </visual>
+        <collision>
+            <origin xyz="0 0 0.05" />
+            <geometry>
+                <cylinder radius="0.3" length="0.1" />
+            </geometry>
+        </collision>
+        <inertial>
+            <origin xyz="0 0 0.05" />
+            <mass value="0.1" />
+            <inertia ixx="0.0023333333333333" ixy="0" ixz="0" iyz="0"
+                iyy=" 0.0023333333333333" izz="0.00075" />
+        </inertial>
+    </link>
+    <joint name=" wheel_base_to_left_wheel" type="continuous">
+        <origin xyz="0 -1 0" rpy="1.57 0 0" />
+        <parent link="wheel_base" />
+        <child link="left_wheel" />
+        <axis xyz=" 0 0 1" />
+    </joint>
+    <link name="right_wheel">
+        <visual>
+            <origin xyz="0 0 -0.05" />
+            <geometry>
+                <cylinder radius="0.3" length="0.1" />
+            </geometry>
+        </visual>
+        <collision>
+            <origin xyz="0 0 -0.05" />
+            <geometry>
+                <cylinder radius="0.3" length="0.1" />
+            </geometry>
+        </collision>
+        <inertial>
+            <origin xyz="0 0 -0.05" />
+            <mass value="0.1" />
+            <inertia ixx="0.0023333333333333" ixy="0" ixz="0" iyz="0"
+                iyy=" 0.0023333333333333" izz="0.00075" />
+        </inertial>
+    </link>
+    <joint name=" wheel_base_to_right_wheel" type="continuous">
+        <origin xyz="0 1 0" rpy="1.57 0 0" />
+        <parent link="wheel_base" />
+        <child link="right_wheel" />
+        <axis xyz=" 0 0 1" />
+    </joint>
+    ------------------------------------------------------------------------------------ rear sphere wheel
+    <link name="rear_wheel">
+        <visual>
+            <geometry>
+                <sphere radius="0.1" />
+            </geometry>
+        </visual>
+        <collision>
+            <geometry>
+                <sphere radius="0.1" />
+            </geometry>
+        </collision>
+        <inertial>
+            <mass value="0.1" />
+            <inertia ixx="0.0004" ixy="0" ixz="0" iyz="0"
+                iyy=" 0.0004" izz="0.0004" />
+        </inertial>
+    </link>
+    <joint name="body_to_rear_wheel" type="continuous">
+        <origin xyz="-1 0 -0.5" />
+        <axis xyz="0 1 0"/>
+        <parent link="body" />
+        <child link="rear_wheel" />
+    </joint>
+    <gazebo>
     <plugin name="model_plugin" filename="libmodel_plugin.so"/>
   </gazebo>
