Commit message: Synchronize model with Controller
Use multi-threading to succeed synchronized communication between model Class and Controller.
Put wind link on base link to avoid torque from drag.

File: urdf/plane.urdf.xacro (robot description, xacro)
@@ -39,5 +39,5 @@
     </link>
     <joint name="bodyToWing" type="revolute">
-        <origin xyz="0 0 0.4" rpy ="0 0 0"/>
+        <origin xyz="0 0 0" rpy ="0 0 0"/>
         <parent link="body" />
         <child link="airfoil" />
