Commit message: Tf_publisher
Add joint_state_publisher and robot_state_publisher
Build some first files for initialized spawning

File: last_letter_2/models/aircraft/plane.urdf.xacro (robot description, xacro)
@@ -136,5 +136,5 @@
         </inertial>
     </link>
-    <joint name=" wheel_base_to_left_wheel" type="continuous">
+    <joint name="wheel_base_to_left_wheel" type="continuous">
         <origin xyz="0 -1 0" rpy="1.57 0 0" />
         <parent link="wheel_base" />
@@ -162,5 +162,5 @@
         </inertial>
     </link>
-    <joint name=" wheel_base_to_right_wheel" type="continuous">
+    <joint name="wheel_base_to_right_wheel" type="continuous">
         <origin xyz="0 1 0" rpy="1.57 0 0" />
         <parent link="wheel_base" />
@@ -194,4 +194,9 @@
     <gazebo>
     <plugin name="model_plugin" filename="libmodel_plugin.so"/>
+    <plugin name="joint_state_publisher" filename="libgazebo_ros_joint_state_publisher.so">
+        <jointName>bodyToWing, body_to_arm, wheel_base_to_left_wheel, wheel_base_to_right_wheel, body_to_rear_wheel </jointName>
+        <robotNamespace>last_letter_2</robotNamespace>
+        <updateRate>100</updateRate>
+    </plugin>
   </gazebo>
 </robot>
