Commit message: Sensors Plugins
Add some of the basic default sensor plugins

File: last_letter_2/config/param/aircrafts/csl_2k19/urdf/model.urdf.xacro (robot description, xacro)
@@ -32,4 +32,9 @@
                         izz="${1/2*body_m*body_r*body_r}" />
         </inertial>
+        <sensor name='my_contact' type='contact'>
+          <contact>
+            <collision>box_collision</collision>
+          </contact>
+        </sensor>
     </link>
     ----------------------------------------------------------------------------  airfoils
@@ -278,12 +283,162 @@
         <child link="rear_wheel" />
     </joint>
+    <joint name="camera_joint" type="revolute">
+    <axis xyz="0 1 0" />
+    <origin xyz="0 ${airfoil_y/2-0.1} -0.1" rpy="0 0 -0.6"/>
+    <parent link="airfoil1"/>
+    <child link="camera_link"/>
+    <limit effort="1000.0" velocity="0.5"/>   ---default limits upper=lower=0
+  </joint>
+  <!-- Camera -->
+  <link name="camera_link">
+    <collision>
+      <origin xyz="0 0 0" rpy="0 0 0"/>
+      <geometry>
+    <box size="0.2 0.2 0.2"/>
+      </geometry>
+    </collision>
+    <visual>
+      <origin xyz="0 0 0" rpy="0 0 0"/>
+      <geometry>
+    <box size="0.2 0.2 0.2"/>
+      </geometry>
+      <material name="red"/>
+    </visual>
+    <inertial>
+      <mass value="1e-5" />
+      <origin xyz="0 0 0" rpy="0 0 0"/>
+      <inertia ixx="1e-6" ixy="0" ixz="0" iyy="1e-6" iyz="0" izz="1e-6" />
+    </inertial>
+  </link>
+  <joint name="hokuyo_joint" type="revolute">
+    <axis xyz="0 1 0" />
+    <origin xyz="${body_h+0.2} 0 0" rpy="0 .2 0"/>
+    <parent link="body_FLU"/>
+    <child link="hokuyo_link"/>
+    <limit effort="1000.0" velocity="0.5"/>   ---default limits upper=lower=0
+  </joint>
+  <!-- Hokuyo Laser -->
+  <link name="hokuyo_link">
+    <collision>
+      <origin xyz="0 0 0" rpy="0 0 0"/>
+      <geometry>
+    <box size="0.1 0.1 0.1"/>
+      </geometry>
+    </collision>
+    <visual>
+      <origin xyz="0 0 0" rpy="0 0 0"/>
+      <geometry>
+        <box size="0.1 0.1 0.1"/>
+      </geometry>
+    </visual>
+    <inertial>
+      <mass value="1e-5" />
+      <origin xyz="0 0 0" rpy="0 0 0"/>
+      <inertia ixx="1e-6" ixy="0" ixz="0" iyy="1e-6" iyz="0" izz="1e-6" />
+    </inertial>
+  </link>
 <!-- model plugins -->
     <gazebo>
-    <plugin name="model_plugin" filename="libmodel_plugin.so"/>
-    <plugin name="joint_state_publisher" filename="libgazebo_ros_joint_state_publisher.so">
-        <jointName>body_FLU_to_airfoil1, body_FLU_to_motor1, motor1_to_axle1, wheel_base_to_left_wheel, wheel_base_to_right_wheel, body_FLU_to_rear_wheel </jointName>
-        <robotNamespace>last_letter_2</robotNamespace>
-        <updateRate>0</updateRate>
-    </plugin>
+        <plugin name="model_plugin" filename="libmodel_plugin.so"/>
+        <plugin name="joint_state_publisher" filename="libgazebo_ros_joint_state_publisher.so">
+            <jointName>body_FLU_to_airfoil1, body_FLU_to_motor1, motor1_to_axle1, wheel_base_to_left_wheel, wheel_base_to_right_wheel, body_FLU_to_rear_wheel, hokuyo_joint, camera_joint </jointName>
+            <robotNamespace>last_letter_2</robotNamespace>
+            <updateRate>0</updateRate>
+        </plugin>
+    </gazebo>
+<!-- camera -->
+  <gazebo reference="camera_link">
+    <sensor type="camera" name="camera1">
+      <update_rate>30.0</update_rate>
+      <camera name="head">
+        <horizontal_fov>1.3962634</horizontal_fov>
+        <image>
+          <width>800</width>
+          <height>800</height>
+          <format>R8G8B8</format>
+        </image>
+        <clip>
+          <near>0.02</near>
+          <far>300</far>
+        </clip>
+        <noise>
+          <type>gaussian</type>
+          <!-- Noise is sampled independently per pixel on each frame.
+               That pixel's noise value is added to each of its color
+               channels, which at that point lie in the range [0,1]. -->
+          <mean>0.0</mean>
+          <stddev>0.007</stddev>
+        </noise>
+      </camera>
+      <plugin name="camera_controller" filename="libgazebo_ros_camera.so">
+        <alwaysOn>true</alwaysOn>
+        <updateRate>0.0</updateRate>
+        <cameraName>rrbot/camera1</cameraName>
+        <imageTopicName>image_raw</imageTopicName>
+        <cameraInfoTopicName>camera_info</cameraInfoTopicName>
+        <frameName>camera_link</frameName>
+        <hackBaseline>0.07</hackBaseline>
+        <distortionK1>0.0</distortionK1>
+        <distortionK2>0.0</distortionK2>
+        <distortionK3>0.0</distortionK3>
+        <distortionT1>0.0</distortionT1>
+        <distortionT2>0.0</distortionT2>
+      </plugin>
+    </sensor>
+  </gazebo>
+ <!-- hokuyo -->
+  <gazebo reference="hokuyo_link">
+    <sensor type="ray" name="head_hokuyo_sensor">
+      <pose>0 0 0 0 0 0</pose>
+      <visualize>true</visualize>
+      <update_rate>40</update_rate>
+      <ray>
+        <scan>
+          <horizontal>
+            <samples>720</samples>
+            <resolution>1</resolution>
+            <min_angle>-1.570796</min_angle>
+            <max_angle>1.570796</max_angle>
+          </horizontal>
+        </scan>
+        <range>
+          <min>0.1</min>
+          <max>30.0</max>
+          <resolution>0.1</resolution>
+        </range>
+        <noise>
+          <type>gaussian</type>
+          <!-- Noise parameters based on published spec for Hokuyo laser
+               achieving "+-30mm" accuracy at range < 10m.  A mean of 0.0m and
+               stddev of 0.01m will put 99.7% of samples within 0.03m of the true
+               reading. -->
+          <mean>0.0</mean>
+          <stddev>0.01</stddev>
+        </noise>
+      </ray>
+      <plugin name="gazebo_ros_head_hokuyo_controller" filename="libgazebo_ros_laser.so">
+        <topicName>/rrbot/laser/scan</topicName>
+        <frameName>hokuyo_link</frameName>
+      </plugin>
+    </sensor>
+  </gazebo>
+   <gazebo reference="body_FLU">
+    <gravity>true</gravity>
+    <sensor name="imu_sensor" type="imu">
+      <always_on>true</always_on>
+      <update_rate>100</update_rate>
+      <visualize>true</visualize>
+      <topic>__default_topic__</topic>
+      <plugin filename="libgazebo_ros_imu_sensor.so" name="imu_plugin">
+        <topicName>imu</topicName>
+        <bodyName>body_FLU</bodyName>
+        <updateRateHZ>10.0</updateRateHZ>
+        <gaussianNoise>0.0</gaussianNoise>
+        <xyzOffset>0 0 0</xyzOffset>
+        <rpyOffset>0 0 0</rpyOffset>
+        <frameName>body_FLU</frameName>
+      </plugin>
+      <pose>0 0 -${body_r+0.01} 0 0 0</pose>
+    </sensor>
   </gazebo>
 </robot>
